File: 0xaxe/0xaxe.kicad_sch (KiCad schematic)
At the start: 6 parts, among them J2 Conn_01x04, J3 Barrel_Jack_Switch

Commit message: rev1.2
Parts:
- F1: Manufacturer 0154005.DR -> 0154.500DR; OrderNr F1228CT-ND -> F1220CT-ND
Other:
- sheet Power ports: added +6.5V; removed none
Changed lines of the file:
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@@
+	(wire
+		(pts
+			(xy 119.38 59.69) (xy 121.92 59.69)
+		)
+		(stroke
+			(width 0)
+			(type default)
+		)
+	)
 	(wire
 		(pts
@@
 			)
 		)
-		(property "Manufacturer" "0154005.DR"
+		(property "Manufacturer" "0154.500DR"
 			(at 72.39 54.61 0)
 			(effects
@@
 			)
 		)
-		(property "OrderNr" "F1228CT-ND"
+		(property "OrderNr" "F1220CT-ND"
 			(at 72.39 54.61 0)
 			(effects
@@
 		)
 	)
+	(symbol
+		(lib_id "mylib7:+6.5V")
+		(at 121.92 59.69 270)
+		(unit 1)
+		(exclude_from_sim no)
+		(in_bom yes)
+		(on_board yes)
+		(dnp no)
+		(fields_autoplaced yes)
+		(property "Reference" "#PWR0490"
+			(at 118.11 59.69 0)
+			(effects
+				(font
+					(size 1.27 1.27)
+				)
+				(hide yes)
+			)
+		)
+		(property "Value" "+6.5V"
+			(at 125.73 59.6899 90)
+			(effects
+				(font
+					(size 1.27 1.27)
+				)
+				(justify left)
+			)
+		)
+		(property "Footprint" ""
+			(at 121.92 59.69 0)
+			(effects
+				(font
+					(size 1.27 1.27)
+				)
+				(hide yes)
+			)
+		)
+		(property "Datasheet" ""
+			(at 121.92 59.69 0)
+			(effects
+				(font
+					(size 1.27 1.27)
+				)
+				(hide yes)
+			)
+		)
+		(property "Description" ""
+			(at 121.92 59.69 0)
+			(effects
+				(font
+					(size 1.27 1.27)
+				)
+				(hide yes)
+			)
+		)
+		(pin "1"
+		)
+		(instances
+			(project "0xaxe"
+				(path "/e63e39d7-6ac0-4ffd-8aa3-1841a4541b55"
+					(reference "#PWR0490")
+					(unit 1)
+				)
+			)
+		)
+	)
 	(sheet
 		(at 134.62 53.34)
@@
 			(effects
 				(font
+					(size 1.27 1.27)
+				)
+				(justify right)
+			)
+		)
+		(pin "+6.5V" output
+			(at 119.38 59.69 0)
+			(effects
+				(font

Commit message: General Update
Other:
- moved on the sheet: D3
Changed lines of the file:
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@@
-	)
-	(junction
-		(at 77.47 20.32)
-		(diameter 0)
-		(color 0 0 0 0)
 	)
 	(junction
@@
 		(color 0 0 0 0)
 	)
+	(junction
+		(at 79.375 20.32)
+		(diameter 0)
+		(color 0 0 0 0)
+	)
 	(wire
 		(pts
@@
 	(wire
 		(pts
-			(xy 87.63 20.32) (xy 77.47 20.32)
+			(xy 71.12 20.32) (xy 79.375 20.32)
 		)
 		(stroke
@@
 	(wire
 		(pts
+			(xy 79.375 20.32) (xy 87.63 20.32)
+		)
+		(stroke
+			(width 0)
+			(type default)
+		)
+	)
+	(wire
+		(pts
 			(xy 158.75 95.25) (xy 171.45 95.25)
 		)
@@
 	(wire
 		(pts
-			(xy 77.47 20.32) (xy 77.47 21.59)
+			(xy 79.375 20.32) (xy 79.375 21.59)
 		)
 		(stroke
@@
 	(wire
 		(pts
-			(xy 77.47 29.21) (xy 77.47 30.48)
+			(xy 79.375 29.21) (xy 79.375 30.48)
 		)
 		(stroke
@@
 		(pts
 			(xy 71.12 25.4) (xy 71.12 30.48)
-		)
-		(stroke
-			(width 0)
-			(type default)
-		)
-	)
-	(wire
-		(pts
-			(xy 77.47 20.32) (xy 71.12 20.32)
 		)
 		(stroke
@@
 	(symbol
 		(lib_id "Diode:5KPxxA")
-		(at 77.47 25.4 270)
+		(at 79.375 25.4 270)
 		(unit 1)
 		(exclude_from_sim no)
@@
 		(dnp no)
 		(property "Reference" "D3"
-			(at 73.025 29.21 0)
+			(at 74.93 29.21 0)
 			(effects
 				(font
@@
 		)
 		(property "Value" "SMBJ5.0A"
-			(at 74.93 22.86 0)
+			(at 76.835 22.86 0)
 			(effects
 				(font
@@
 		)
 		(property "Footprint" "Diode_SMD:D_SMB"
-			(at 72.39 25.4 0)
+			(at 74.295 25.4 0)
 			(effects
 				(font
@@
 		)
 		(property "Datasheet" ""
-			(at 77.47 24.13 0)
+			(at 79.375 24.13 0)
 			(effects
 				(font
@@
 		)
 		(property "Description" ""
-			(at 77.47 25.4 0)
+			(at 79.375 25.4 0)
 			(effects
 				(font
@@
 		)
 		(property "Distributor" "D"
-			(at 77.47 25.4 0)
+			(at 79.375 25.4 0)
 			(effects
 				(font
@@
 		)
 		(property "Manufacturer" "SMBJ5.0A"
-			(at 77.47 25.4 0)
+			(at 79.375 25.4 0)
 			(effects
 				(font
@@
 		)
 		(property "OrderNr" "SMBJ5.0ALFCT-ND"
-			(at 77.47 25.4 0)
+			(at 79.375 25.4 0)
 			(effects
 				(font
@@
 	(symbol
 		(lib_id "power:GND")
-		(at 77.47 30.48 0)
+		(at 79.375 30.48 0)
 		(unit 1)
 		(exclude_from_sim no)
@@
 		(dnp no)
 		(property "Reference" "#PWR012"
-			(at 77.47 36.83 0)
+			(at 79.375 36.83 0)
 			(effects
 				(font
@@
 		)
 		(property "Value" "GND"
-			(at 77.597 34.8742 0)
+			(at 79.502 34.8742 0)
 			(effects
 				(font
@@
 		)
 		(property "Footprint" ""
-			(at 77.47 30.48 0)
+			(at 79.375 30.48 0)
 			(effects
 				(font
@@
 		)
 		(property "Datasheet" ""
-			(at 77.47 30.48 0)
+			(at 79.375 30.48 0)
 			(effects
 				(font
@@
 		)
 		(property "Description" ""
-			(at 77.47 30.48 0)
-			(effects
-				(font
+			(at 79.375 30.48 0)
+			(effects
+				(font

Commit message: fixed couple of things
Other:
- sheet flex ports: added none; removed +3V3_IF, GND_IF
- moved on the sheet: D3, F1, J2, J3
