File: 0xaxe/flex3.kicad_sch (KiCad schematic)
At the start: 89 parts, among them U39 MCP1824T-1802E, U7001 25MHz, U7003 NCP114ASN080T1G, U7004 ADUM141E0BRZ-RL7, U7005 +0V8, U7006 +0V8, U7007 BM1366_mode1, U7008 +0V8, U7009 +0V8, U7010 +0V8, U7011 +0V8, U7012 +0V8, U7013 +0V8, U7014 +0V8, U7015 +0V8, U7016 +0V8, U7017 +0V8, U7018 BM1366_mode1, U7019 +0V8, U7020 +0V8, U7021 BM1366_mode1, U7022 +0V8, U7024 +0V8, U7025 BM1366_mode1, U7026 +0V8

Commit message: op levelshifter
Parts:
- removed C7010, C7011: 100n, Capacitor_SMD:C_0805_2012Metric, symbol Device:C
- removed U7004: ADUM141E0BRZ-RL7, Package_SO:SOIC-16_3.9x9.9mm_P1.27mm, symbol Isolator:ADuM1411
- added C167: 0.1uF, Capacitor_SMD:C_0805_2012Metric, symbol Device:C
- added C168: 1uF, Capacitor_SMD:C_0805_2012Metric, symbol Device:C
- added C288, C289, C290, C291: 100pF, Capacitor_SMD:C_0805_2012Metric, symbol Device:C
- added R100, R101, R89, R90, R92, R93, R97, R98: 10k, Resistor_SMD:R_0805_2012Metric, symbol Device:R
- added R102, R103, R104, R88, R91, R94, R95, R96, R99: 1k, Resistor_SMD:R_0805_2012Metric, symbol Device:R
- added U66: TLV3544, Package_SO:SOIC-14_3.9x8.7mm_P1.27mm, symbol bitaxe:TLV3544
- renumbered C7002 to C159, C7003 to C160, C7004 to C161, C7005 to C162, C7006 to C163, C7007 to C164, C7009 to C166, C7012 to C169, C7013 to C170, C7014 to C171, C7015 to C172, C7016 to C173, C7017 to C174, C7018 to C175, C7019 to C176, C7020 to C177, C7021 to C178, C7022 to C179, C7023 to C180, C7024 to C181, C7025 to C182, C7026 to C183, C7027 to C184, C7028 to C185, C7029 to C186, C7030 to C187, C7031 to C188, C7032 to C189, C7033 to C190, C7034 to C191, C7035 to C192, C7036 to C193, C7037 to C194, C7038 to C195, C7039 to C196, C7040 to C197, C7041 to C198, C7042 to C199, C7043 to C200, C7044 to C201, C7045 to C202, C7046 to C203, C7047 to C204, C7048 to C205, C7049 to C206, C7050 to C207, C7051 to C208, C7052 to C209, C7053 to C210, C7054 to C211, C7055 to C212, C7057 to C213, C7058 to C214, C7059 to C215, C7060 to C216, C7061 to C217, R7003 to R50, R7004 to R51, R7005 to R52, R7006 to R53, U7001 to U63, U7003 to U65, U7005 to U67, U7006 to U68, U7007 to U69, U7008 to U70, U7009 to U71, U7010 to U72, U7011 to U73, U7012 to U74, U7013 to U75, U7014 to U76, U7015 to U77, U7016 to U78, U7017 to U79, U7018 to U80, U7019 to U81, U7020 to U82, U7021 to U83, U7022 to U84, U7024 to U85, U7025 to U86, U7026 to U87
Connections:
- net +6.5V: now also C167.2, C168.2, U66.4 (V+)
- net BI: now also R101.1
- net CI: now also R90.1
- net GND_2: now also R88.2, R91.2, R96.2, R99.2
- net NRSTI: now also R93.1
- net NRSTO: now also C289.2, R95.1, U66.7; no longer U69.5 (NRSTI)
- net RO: now also R104.1
- net CLKI: no longer names the net of U63.3 (Out)
- net CLKI: no longer U69.8 (CLKI)
- new net: R89.1, R90.2, U66.3 (+)
- new net: R92.2, R93.2, U66.5 (+)
- new net: C289.1, R91.1, R95.2, U66.6 (-)
- new net: R97.2, R98.2, U66.12 (+)
- new net: R100.2, R101.2, U66.10 (+)
- new net: C291.1, R103.2, R99.1, U66.9 (-)
- new net: C288.1, R88.1, R94.2, U66.2 (-)
- new net: C290.2, R102.1, R104.2, U66.14
- new net: C290.1, R102.2, R96.1, U66.13 (-)
- new net BI_2: C291.2, R103.1, U66.8
- new net CI_2: C288.2, R94.1, U66.1
- new net GND: C167.1, C168.1, U66.11 (V-)
- new net I_CLKI: U69.8 (CLKI)
- new net I_NRSTI: U69.5 (NRSTI)
- new net RO_2: R98.1
- new net VDD_2: R100.1, R89.2, R92.1
- new net VDD_REF_I: R97.1
- no-connect marks 21 -> 19
Other:
- note added: "25MHz Osc for CLKI"
- note added: "Levelshift of input signals to own voltage domain"
- note added: "OPAMP Bypass"
- moved on the sheet: C159, C160, C161, C162, C163, C164, C166, C169, C170, C171, C172, C173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

Commit message: General Update
Parts:
- U67, U68, U70, U71, U72, U73, U74, U75, U76, U77, U78, U79, U81, U82, U84, U85, U87: value +0V8 -> +0V8_2
Other:
- moved on the sheet: C170, C171, C173, C174, C175, C176, C178, C179, C180, C181, C182, C184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

Commit message: fixed couple of things
Connections:
- net BI is gone; now on net BI_2: R101.1
- net CI is gone; now on net CI_2: R90.1
- net I_CLKI is gone; now on net I_CLKI_2: U69.8 (CLKI)
- net NRSTO is gone; now on net NRSTO_2: C289.2, R95.1, U66.7
- net RO is gone; now on net RO_2: R104.1
- net VDD_2 is gone; now on net +1V2_2: R100.1, R89.2, R92.1
- net BI_2: no longer C291.2, R103.1, U66.8
- net CI_2: no longer C288.2, R94.1, U66.1
- net RO_2: no longer R98.1
- net I_CLKI_2: now reaches U63.3 (Out)
- net BO renamed BO_2
- net CO renamed CO_2
- net I_BI renamed I_BI_2
- net I_BI_2: now also C291.2, R103.1, U66.8
- net I_CI renamed I_CI_2
- net I_CI_2: now also C288.2, R94.1, U66.1
- net I_NRSTI renamed NRSTO_2
- net I_RO renamed I_RO_2
- net I_RO_2: now also R98.1
- net NRSTI renamed NRSTI_2
- net RI renamed RI_2
- net VDD_REF_I renamed VDD_REF_I_2
Other:
- moved on the sheet: C159, C162, C163, C166, C167, C169, C170, C171, C173, C174, C175, C176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

Commit message: Layout update
Layout with OP
Parts:
- removed R100, R101, R89, R90, R92, R93, R97, R98: 10k, Resistor_SMD:R_0805_2012Metric, symbol Device:R
- removed R102, R103, R104, R88, R91, R94, R95, R96, R99: 1k, Resistor_SMD:R_0805_2012Metric, symbol Device:R
- added RN10, RN11, RN12, RN9: 10k, EXB-28V103JX:EXB28V_PAN, symbol Device:R_Network04_Split
- U69, U80, U83, U86: footprint qaxe:BM1366 -> bitvein:BM1366
Connections:
- net +1V2_2: now also RN10.1 (R1), RN12.4 (R2.2), RN9.8 (R4.2)
- net BI_2: now also RN12.5 (R2.2)
- net CI_2: now also RN9.1 (R1)
- net GND_2: now also RN10.4 (R2.2), RN11.4 (R2.2), RN12.1 (R1), RN9.5 (R2.2)
- net I_BI_2: now also RN12.8 (R4.2)
- net I_CI_2: now also RN9.4 (R2.2)
- net I_RO_2: now also RN11.8 (R4.2)
- net NRSTI_2: now also RN10.8 (R4.2)
- net NRSTO_2: now also RN10.5 (R2.2)
- net RO_2: now also C290.2, U66.14, RN11.5 (R2.2)
- net VDD_REF_I_2: now also RN11.1 (R1)
- net at U66.3 (+): now also RN9.2 (R1.2), RN9.7 (R2.2)
- net at U66.5 (+): now also RN10.2 (R1.2), RN10.7 (R2.2)
- net at C289.1, U66.6 (-): now also RN10.3 (R2.2), RN10.6 (R3.2)
- net at U66.12 (+): now also RN11.2 (R1.2), RN11.7 (R2.2)
- net at U66.10 (+): now also RN12.3 (R2.2), RN12.6 (R3.2)
- net at C291.1, U66.9 (-): now also RN12.2 (R1.2), RN12.7 (R2.2)
- net at C288.1, U66.2 (-): now also RN9.3 (R2.2), RN9.6 (R3.2)
- net at C290.1, U66.13 (-): now also RN11.3 (R2.2), RN11.6 (R3.2)
