File: 0xaxe/flex3.kicad_sch (KiCad schematic)
At the start: 89 parts, among them U39 MCP1824T-1802E, U7001 25MHz, U7003 NCP114ASN080T1G, U7004 ADUM141E0BRZ-RL7, U7005 +0V8, U7006 +0V8, U7007 BM1366_mode1, U7008 +0V8, U7009 +0V8, U7010 +0V8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

Commit message: rev1.2
Connections:
- net +5V renamed +6.5V
Changed lines of the file:
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@@
 	)
 	(symbol
+		(lib_id "mylib7:+6.5V")
+		(at 87.63 184.15 0)
+		(unit 1)
+		(exclude_from_sim no)
+		(in_bom yes)
+		(on_board yes)
+		(dnp no)
+		(fields_autoplaced yes)
+		(property "Reference" "#PWR0155"
+			(at 87.63 187.96 0)
+			(effects
+				(font
+					(size 1.27 1.27)
+				)
+				(hide yes)
+			)
+		)
+		(property "Value" "+6.5V"
+			(at 87.63 179.07 0)
+			(effects
+				(font
+					(size 1.27 1.27)
+				)
+			)
+		)
+		(property "Footprint" ""
+			(at 87.63 184.15 0)
+			(effects
+				(font
+					(size 1.27 1.27)
+				)
+				(hide yes)
+			)
+		)
+		(property "Datasheet" ""
+			(at 87.63 184.15 0)
+			(effects
+				(font
+					(size 1.27 1.27)
+				)
+				(hide yes)
+			)
+		)
+		(property "Description" ""
+			(at 87.63 184.15 0)
+			(effects
+				(font
+					(size 1.27 1.27)
+				)
+				(hide yes)
+			)
+		)
+		(pin "1"
+		)
+		(instances
+			(project "0xaxe"
+				(path "/e63e39d7-6ac0-4ffd-8aa3-1841a4541b55/84d407d0-bd71-403d-bc5c-679b63d0a5ac/05480cd1-7be0-4875-99b4-e3dcbd164eca"
+					(reference "#PWR0155")
+					(unit 1)
+				)
+			)
+		)
+	)
+	(symbol
 		(lib_id "mylib7:GND_2")
 		(at 298.45 203.2 0)
@@
 					(unit 1)
 				)
-			)
-		)
-	)
-	(symbol
-		(lib_id "power:+5V")
-		(at 87.63 184.15 0)
-		(unit 1)
-		(exclude_from_sim no)
-		(in_bom yes)
-		(on_board yes)
-		(dnp no)
-		(fields_autoplaced yes)
-		(property "Reference" "#PWR0155"
-			(at 87.63 187.96 0)
-			(effects
-				(font
-					(size 1.27 1.27)
-				)
-				(hide yes)
-			)
-		)
-		(property "Value" "+5V"
-			(at 87.63 179.07 0)
-			(effects
-				(font
-					(size 1.27 1.27)
-				)
-			)
-		)
-		(property "Footprint" ""
-			(at 87.63 184.15 0)
-			(effects
-				(font
-					(size 1.27 1.27)
-				)
-				(hide yes)
-			)
-		)
-		(property "Datasheet" ""
-			(at 87.63 184.15 0)
-			(effects
-				(font
-					(size 1.27 1.27)
-				)
-				(hide yes)
-			)
-		)
-		(property "Description" "Power symbol creates a global label with name \"+5V\""
-			(at 87.63 184.15 0)
-			(effects
-				(font
-					(size 1.27 1.27)
-				)
-				(hide yes)
-			)
-		)
-		(pin "1"
-		)
-		(instances
-			(project "0xaxe"
-				(path "/e63e39d7-6ac0-4ffd-8aa3-1841a4541b55/84d407d0-bd71-403d-bc5c-679b63d0a5ac/05480cd1-7be0-4875-99b4-e3dcbd164eca"
-					(reference "#PWR0155")
-					(unit 1)
-				)

Commit message: push
Parts:
- U7004: footprint Package_SO:SOIC-16_3.9x9.9mm_P1.27mm -> Package_SO:QSOP-16_3.9x4.9mm_P0.635mm; Manufacturer ADUM141E0BRZ-RL7 -> ADUM141D1BRQZ; OrderNr 505-ADUM141E0BRZ-RL7CT-ND -> ADUM141D1BRQZ-ND
Changed lines of the file:
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@@
 			)
 		)
-		(property "Footprint" "Package_SO:SOIC-16_3.9x9.9mm_P1.27mm"
+		(property "Footprint" "Package_SO:QSOP-16_3.9x4.9mm_P0.635mm"
 			(at 105.41 151.13 0)
 			(effects
@@
 			)
 		)
-		(property "Manufacturer" "ADUM141E0BRZ-RL7"
+		(property "Manufacturer" "ADUM141D1BRQZ"
 			(at 105.41 133.35 0)
 			(effects
@@
 			)
 		)
-		(property "OrderNr" "505-ADUM141E0BRZ-RL7CT-ND"
+		(property "OrderNr" "ADUM141D1BRQZ-ND"
 			(at 105.41 133.35 0)
 			(effects
