File: 0xaxe/flex.kicad_sch (KiCad schematic)
At the start: 37 parts, among them U4 INA500DCK, U5 INA500DCK, U6 INA500DCK, U7 INA500DCK, U8 ISL21080CIH315Z-TK, U9 LM339

Commit message: fixed BOM
Parts:
- C9: Distributor D -> (none); Manufacturer CAY16-1002F4LF -> (none); OrderNr CAY16-1002F4LFCT-ND -> (none)
Changed lines of the file:
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@@
 			)
 		)
-		(property "Distributor" "D"
+		(property "Distributor" ""
 			(at 289.56 66.04 0)
 			(effects
@@
 			)
 		)
-		(property "Manufacturer" "CAY16-1002F4LF"
+		(property "Manufacturer" ""
 			(at 289.56 66.04 0)
 			(effects
@@
 			)
 		)
-		(property "OrderNr" "CAY16-1002F4LFCT-ND"
+		(property "OrderNr" ""
 			(at 289.56 66.04 0)
 			(effects
@@
 			)
 		)
-		(property "Distributor" "D"
+		(property "Distributor" ""
 			(at 308.61 66.04 0)
 			(effects
@@
 			)
 		)
-		(property "Manufacturer" "CAY16-1002F4LF"
+		(property "Manufacturer" ""
 			(at 308.61 66.04 0)
 			(effects
@@
 			)
 		)
-		(property "OrderNr" "CAY16-1002F4LFCT-ND"
+		(property "OrderNr" ""
 			(at 308.61 66.04 0)
 			(effects
@@
 			)
 		)
-		(property "Distributor" "D"
+		(property "Distributor" ""
 			(at 317.5 66.04 0)
 			(effects
@@
 			)
 		)
-		(property "Manufacturer" "CAY16-1002F4LF"
+		(property "Manufacturer" ""
 			(at 317.5 66.04 0)
 			(effects
@@
 			)
 		)
-		(property "OrderNr" "CAY16-1002F4LFCT-ND"
+		(property "OrderNr" ""
 			(at 317.5 66.04 0)
 			(effects

Commit message: fixed level shifter, added optional headers for future extensions
Parts:
- C9: Distributor (none) -> D; Manufacturer (none) -> CAY16-1002F4LF; OrderNr (none) -> CAY16-1002F4LFCT-ND
Changed lines of the file:
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@@
 			)
 		)
-		(property "Distributor" ""
+		(property "Distributor" "D"
 			(at 289.56 66.04 0)
 			(effects
@@
 			)
 		)
-		(property "Manufacturer" ""
+		(property "Manufacturer" "CAY16-1002F4LF"
 			(at 289.56 66.04 0)
 			(effects
@@
 			)
 		)
-		(property "OrderNr" ""
+		(property "OrderNr" "CAY16-1002F4LFCT-ND"
 			(at 289.56 66.04 0)
 			(effects
@@
 			)
 		)
-		(property "Distributor" ""
+		(property "Distributor" "D"
 			(at 308.61 66.04 0)
 			(effects
@@
 			)
 		)
-		(property "Manufacturer" ""
+		(property "Manufacturer" "CAY16-1002F4LF"
 			(at 308.61 66.04 0)
 			(effects
@@
 			)
 		)
-		(property "OrderNr" ""
+		(property "OrderNr" "CAY16-1002F4LFCT-ND"
 			(at 308.61 66.04 0)
 			(effects
@@
 			)
 		)
-		(property "Distributor" ""
+		(property "Distributor" "D"
 			(at 317.5 66.04 0)
 			(effects
@@
 			)
 		)
-		(property "Manufacturer" ""
+		(property "Manufacturer" "CAY16-1002F4LF"
 			(at 317.5 66.04 0)
 			(effects
@@
 			)
 		)
-		(property "OrderNr" ""
+		(property "OrderNr" "CAY16-1002F4LFCT-ND"
 			(at 317.5 66.04 0)
 			(effects
