File: 0xaxe/flex.kicad_sch (KiCad schematic)
At the start: 47 parts, among them U4 INA500DCK, U5 INA500DCK, U6 INA500DCK, U7 INA500DCK, U8 ISL21080CIH315Z-TK, U9 LM339

Commit message: rev1.2
Parts:
- removed R36, R37, R42, R43, R48, R49, R54, R55: 1, Resistor_SMD:R_2512_6332Metric, symbol Device:R_Small

Commit message: op levelshifter
Parts:
- removed C9 (x3): 10µ/50V, Capacitor_SMD:C_1206_3216Metric, symbol Device:C
- added R105: 22, Resistor_SMD:R_0805_2012Metric, symbol Device:R
- R9: value 22 -> 10k
Connections:
- net BO_0 is gone; now on net GND: R9.2
- net BO_1 is gone; now on net flex2/BO: R11.2
- net BO_2 is gone; now on net flex3/BO: R13.2
- net CO_0 is gone; now on net flex4/BO: R10.2
- net CO_1 is gone; now on net flex2/CO: R12.2
- net CO_2 is gone; now on net flex3/CO: R14.2
- net RI_2 is gone; now on net flex4/RI: R8.1
- net flex4/RO is gone; now on net flex3/RO: R8.2
- net flex1/BO: no longer R9.1
- net flex1/CO: no longer R10.1
- net flex2/BO: no longer R11.1
- net flex2/CO: no longer R12.1
- net flex2/RO: now also R7.2; no longer R6.2
- net flex3/BO: no longer R13.1
- net flex3/CO: no longer R14.1
- net flex3/RO: no longer R7.2
- net flex4/CO: now also R105.2
- net RI_0 renamed flex2/RI
- net RI_1 renamed flex3/RI
- new net flex1/BI: R11.1
- new net flex1/CI: R12.1
- new net flex1/RO: R6.2
- new net flex2/BI: R13.1
- new net flex2/CI: R14.1
- new net flex3/BI: R10.1
- new net flex3/CI: R105.1
- new net flex4/BI: R9.1
- no-connect marks 6 -> 5
Other:
- sheet flex1 ports: added GND_1, VDD_1, VDD_REF_I, VDD_REF_O; removed +1.8V_OUT, +1V2, GND, GND_IF, GND_OUT, V_IF
- sheet flex2 ports: added GND_1, VDD_1, VDD_REF_I, VDD_REF_O; removed +1.8V_OUT, +1V2, GND, GND_IF, GND_OUT, V_IF
- sheet flex3 ports: added GND_2, VDD_2, VDD_REF_I, VDD_REF_O; removed +1.8V_OUT, +1V2, GND, GND_IF, GND_OUT, V_IF
- sheet flex4 ports: added GND_3, VDD_3, VDD_REF_O; removed +1.8V_OUT, +1V2, GND, GND_IF, GND_OUT, V_IF
- moved on the sheet: R11, R12, R13, R14, R6, R7, R8

Commit message: General Update
Connections:
- net flex1/BI renamed BO_1
- net flex1/CI renamed CO_1
- net flex2/BI renamed BO_2
- net flex2/CI renamed CO_2
- net flex2/RI renamed RI_1
- net flex3/BI renamed BO_3
- net flex3/CI renamed CO_3
- net flex3/RI renamed RI_2
- net flex4/RI renamed RI_3
Changed lines of the file:
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@@
 		)
 	)
+	(label "NRSTO_1"
+		(at 123.19 96.52 0)
+		(fields_autoplaced yes)
+		(effects
+			(font
+				(size 1.27 1.27)
+			)
+			(justify left bottom)
+		)
+	)
+	(label "NRSTO_2"
+		(at 123.19 135.89 0)
+		(fields_autoplaced yes)
+		(effects
+			(font
+				(size 1.27 1.27)
+			)
+			(justify left bottom)
+		)
+	)
+	(label "BO_1"
+		(at 121.92 93.98 0)
+		(fields_autoplaced yes)
+		(effects
+			(font
+				(size 1.27 1.27)
+			)
+			(justify left bottom)
+		)
+	)
 	(label "+1V2"
 		(at 175.26 215.9 0)
@@
 		)
 	)
+	(label "CO_2"
+		(at 119.38 128.27 0)
+		(fields_autoplaced yes)
+		(effects
+			(font
+				(size 1.27 1.27)
+			)
+			(justify left bottom)
+		)
+	)
+	(label "CO_3"
+		(at 119.38 170.18 0)
+		(fields_autoplaced yes)
+		(effects
+			(font
+				(size 1.27 1.27)
+			)
+			(justify left bottom)
+		)
+	)
+	(label "BO_2"
+		(at 121.92 133.35 0)
+		(fields_autoplaced yes)
+		(effects
+			(font
+				(size 1.27 1.27)
+			)
+			(justify left bottom)
+		)
+	)
+	(label "NRSTO_3"
+		(at 123.19 177.8 0)
+		(fields_autoplaced yes)
+		(effects
+			(font
+				(size 1.27 1.27)
+			)
+			(justify left bottom)
+		)
+	)
 	(label "2.5V"
 		(at 264.16 68.58 0)
@@
 		)
 	)
+	(label "BO_3"
+		(at 121.92 175.26 0)
+		(fields_autoplaced yes)
+		(effects
+			(font
+				(size 1.27 1.27)
+			)
+			(justify left bottom)
+		)
+	)
+	(label "CO_1"
+		(at 119.38 88.9 0)
+		(fields_autoplaced yes)
+		(effects
+			(font
+				(size 1.27 1.27)
+			)
+			(justify left bottom)
+		)
+	)
+	(label "VDD_REF_3"
+		(at 124.46 180.34 0)
+		(fields_autoplaced yes)
+		(effects
+			(font
+				(size 1.27 1.27)
+			)
+			(justify left bottom)
+		)
+	)
+	(label "RI_1"
+		(at 120.65 91.44 0)
+		(fields_autoplaced yes)
+		(effects
+			(font
+				(size 1.27 1.27)
+			)
+			(justify left bottom)
+		)
+	)
+	(label "RI_3"
+		(at 120.65 172.72 0)
+		(fields_autoplaced yes)
+		(effects
+			(font
+				(size 1.27 1.27)
+			)
+			(justify left bottom)
+		)
+	)
+	(label "VDD_REF_1"
+		(at 124.46 99.06 0)
+		(fields_autoplaced yes)
+		(effects
+			(font
+				(size 1.27 1.27)
+			)
+			(justify left bottom)
+		)
+	)
+	(label "RI_2"
+		(at 120.65 130.81 0)
+		(fields_autoplaced yes)
+		(effects
+			(font
+				(size 1.27 1.27)
+			)
+			(justify left bottom)
+		)
+	)
+	(label "VDD_REF_2"
+		(at 124.46 138.43 0)
+		(fields_autoplaced yes)
+		(effects
+			(font
+				(size 1.27 1.27)
+			)
+			(justify left bottom)
+		)
+	)
 	(global_label "V3_G2"
 		(shape passive)
@@
 		(dnp no)
 		(property "Reference" "R8"
-			(at 123.825 171.45 90)
+			(at 132.715 171.45 90)
 			(effects
 				(font
@@
 		(dnp no)
 		(property "Reference" "R6"
-			(at 123.825 90.17 90)
+			(at 132.715 90.17 90)
 			(effects
 				(font
@@
 		(dnp no)
 		(property "Reference" "R7"
-			(at 123.825 129.54 90)
+			(at 132.715 129.54 90)
 			(effects
 				(font

Commit message: fixed couple of things
Connections:
- net BO_1 renamed flex1/BI_0
- net BO_2 renamed flex2/BI_1
- net BO_3 renamed flex3/BI_2
- net CO_1 renamed flex1/CI_0
- net CO_2 renamed flex2/CI_1
- net CO_3 renamed flex3/CI_2
- net RI_1 renamed flex2/RI_1
- net RI_2 renamed flex3/RI_2
- net RI_3 renamed flex4/RI_3
- net flex1/RO renamed flex1/RO_0
- net flex2/BO renamed flex2/BO_1
- net flex2/CO renamed flex2/CO_1
- net flex2/RO renamed flex2/RO_1
- net flex3/BO renamed flex3/BO_2
- net flex3/CO renamed flex3/CO_2
- net flex3/RO renamed flex3/RO_2
- net flex4/BI renamed flex4/BI_3
- net flex4/BO renamed flex4/BO_3
- net flex4/CO renamed flex4/CO_3
- no-connect marks 5 -> 0
Other:
- sheet flex1 ports: added BI_0, CI_0, GND_0, NRSTI_0, RO_0, VDD_0, VDD_REF_I_0; removed BI, BO, CI, CO, GND_1, NRSTI, NRSTO, RI, RO, VDD_1, VDD_REF_I, VDD_REF_O
- sheet flex2 ports: added BI_1, BO_1, CI_1, CO_1, NRSTI_1, NRSTO_1, RI_1, RO_1, VDD_REF_I_1, VDD_REF_O_1; removed BI, BO, CI, CO, NRSTI, NRSTO, RI, RO, VDD_REF_I, VDD_REF_O
- sheet flex3 ports: added BI_2, BO_2, CI_2, CO_2, NRSTI_2, NRSTO_2, RI_2, RO_2, VDD_REF_I_2, VDD_REF_O_2; removed BI, BO, CI, CO, NRSTI, NRSTO, RI, RO, VDD_REF_I, VDD_REF_O
- sheet flex4 ports: added BI_3, BO_3, CI_3, CO_3, NRSTI_3, NRSTO_3, RI_3, RO_3, VDD_REF_O_3; removed BI, BO, CI, CO, NRSTI, NRSTO, RI, RO, VDD_REF_O

Commit message: fixed bom
Parts:
- JP3: now left out of the parts list
Changed lines of the file:
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@@
 		(unit 1)
 		(exclude_from_sim no)
-		(in_bom yes)
+		(in_bom no)
 		(on_board yes)
 		(dnp no)
