File: 0xaxe/flex4.kicad_sch (KiCad schematic)
At the start: 89 parts, among them U10 +0V8, U11 +0V8, U12 +0V8, U13 +0V8, U14 +0V8, U15 +0V8, U16 +0V8, U17 +0V8, U18 +0V8, U19 BM1366_mode1, U2 25MHz, U20 +0V8, U21 +0V8, U22 BM1366_mode1, U23 +0V8, U25 +0V8, U26 BM1366_mode1, U27 +0V8, U4 NCP114ASN080T1G, U5 ADUM141E0BRZ-RL7, U6 +0V8, U64 MCP1824T-1802E, U7 +0V8, U8 BM1366_mode1, U9 +0V8

Commit message: op levelshifter
Parts:
- removed C10, C11: 100n, Capacitor_SMD:C_0805_2012Metric, symbol Device:C
- removed U5: ADUM141E0BRZ-RL7, Package_SO:SOIC-16_3.9x9.9mm_P1.27mm, symbol Isolator:ADuM1411
- renumbered C2 to C219, C3 to C220, C4 to C221, C5 to C222, C6 to C223, C7 to C224, C9 to C226, C12 to C229, C13 to C230, C14 to C231, C15 to C232, C16 to C233, C17 to C234, C18 to C235, C19 to C236, C20 to C237, C21 to C238, C22 to C239, C62 to C240, C24 to C241, C25 to C242, C26 to C243, C27 to C244, C28 to C245, C29 to C246, C30 to C247, C31 to C248, C32 to C249, C33 to C250, C34 to C251, C35 to C252, C36 to C253, C37 to C254, C38 to C255, C39 to C256, C40 to C257, C41 to C258, C42 to C259, C43 to C260, C44 to C261, C56 to C262, C46 to C263, C47 to C264, C48 to C265, C49 to C266, C50 to C267, C51 to C268, C52 to C269, C53 to C270, C54 to C271, C55 to C272, C57 to C273, C58 to C274, C59 to C275, C60 to C276, C61 to C277, R3 to R56, R4 to R57, R5 to R58, R6 to R59, U14 to U100, U15 to U101, U16 to U102, U17 to U103, U18 to U104, U19 to U105, U20 to U106, U21 to U107, U22 to U108, U23 to U109, U25 to U110, U26 to U111, U27 to U112, U2 to U88, U4 to U90, U6 to U92, U7 to U93, U8 to U94, U9 to U95, U10 to U96, U11 to U97, U12 to U98, U13 to U99
Connections:
- net I_BI is gone; now on net BI: U94.6 (BI)
- net I_CI is gone; now on net CI: U94.9 (CI)
- net I_RO is gone; now on net RO: U94.7 (RO)
- net NRSTI: now also U94.5 (NRSTI)
- net NRSTO: now also U111.24 (NRSTO); no longer U94.5 (NRSTI)
- net CLKI renamed I_CLKI
- no-connect marks 21 -> 18
Other:
- note added: "+0V8 LDO"
- note added: "+1V8 LDO"
- note added: "25MHz Osc for CLKI"
- moved on the sheet: C105, C158, C219, C220, C221, C222, C223, C224, C226, C229, C230, C231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

Commit message: General Update
Parts:
- U100, U101, U102, U103, U104, U106, U107, U109, U110, U112, U92, U93, U95, U96, U97, U98, U99: value +0V8 -> +0V8_3
Other:
- note added: "+0V8_3 LDO"
- note removed: "+0V8 LDO"
Changed lines of the file:
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@@
 	(wire
 		(pts
-			(xy 351.79 77.47) (xy 373.38 77.47)
-		)
-		(stroke
-			(width 0)
-			(type default)
-		)
-	)
-	(wire
-		(pts
 			(xy 179.07 173.99) (xy 179.07 175.26)
 		)
@@
 	(wire
 		(pts
+			(xy 351.79 77.47) (xy 373.38 77.47)
+		)
+		(stroke
+			(width 0)
+			(type default)
+		)
+	)
+	(wire
+		(pts
 			(xy 156.21 182.88) (xy 156.21 184.15)
 		)
@@
 		)
 	)
-	(text "+0V8 LDO"
+	(text "+0V8_3 LDO"
 		(exclude_from_sim no)
 		(at 52.07 216.408 0)
@@
 			)
 		)
-		(property "Value" "+0V8"
+		(property "Value" "+0V8_3"
 			(at 156.21 170.815 90)
 			(effects
@@
 			)
 		)
-		(property "Value" "+0V8"
+		(property "Value" "+0V8_3"
 			(at 280.035 87.63 90)
 			(effects
@@
 			)
 		)
-		(property "Value" "+0V8"
+		(property "Value" "+0V8_3"
 			(at 179.07 170.815 90)
 			(effects
@@
 			)
 		)
-		(property "Value" "+0V8"
+		(property "Value" "+0V8_3"
 			(at 162.56 170.815 90)
 			(effects
@@
 			)
 		)
-		(property "Value" "+0V8"
+		(property "Value" "+0V8_3"
 			(at 197.485 87.63 90)
 			(effects
@@
 			)
 		)
-		(property "Value" "+0V8"
+		(property "Value" "+0V8_3"
 			(at 307.975 87.63 90)
 			(effects
@@
 			)
 		)
-		(property "Value" "+0V8"
+		(property "Value" "+0V8_3"
 			(at 361.315 87.63 90)
 			(effects
@@
 			)
 		)
-		(property "Value" "+0V8"
+		(property "Value" "+0V8_3"
 			(at 69.85 225.425 90)
 			(effects
@@
 			)
 		)
-		(property "Value" "+0V8"
+		(property "Value" "+0V8_3"
 			(at 144.145 87.63 90)
 			(effects
@@
 			)
 		)
-		(property "Value" "+0V8"
+		(property "Value" "+0V8_3"
 			(at 226.695 87.63 90)
 			(effects
@@
 			)
 		)
-		(property "Value" "+0V8"
+		(property "Value" "+0V8_3"
 			(at 190.5 170.815 90)
 			(effects
@@
 			)
 		)
-		(property "Value" "+0V8"
+		(property "Value" "+0V8_3"
 			(at 195.58 170.815 90)
 			(effects
@@
 			)
 		)
-		(property "Value" "+0V8"
+		(property "Value" "+0V8_3"
 			(at 116.205 87.63 90)
 			(effects
@@
 			)
 		)
-		(property "Value" "+0V8"
+		(property "Value" "+0V8_3"
 			(at 62.865 87.63 90)
 			(effects
@@
 			)
 		)
-		(property "Value" "+0V8"
+		(property "Value" "+0V8_3"
 			(at 173.99 170.815 90)
 			(effects
@@
 			)
 		)
-		(property "Value" "+0V8"
+		(property "Value" "+0V8_3"
 			(at 167.64 170.815 90)
 			(effects
@@
 			)
 		)
-		(property "Value" "+0V8"
+		(property "Value" "+0V8_3"
 			(at 184.15 170.815 90)
 			(effects

Commit message: fixed couple of things
Connections:
- net BI renamed BI_3
- net BO renamed BO_3
- net CI renamed CI_3
- net CO renamed CO_3
- net I_CLKI renamed I_CLKI_3
- net NRSTI renamed NRSTI_3
- net NRSTO renamed NRSTO_3
- net RI renamed RI_3
- net RO renamed RO_3
Other:
- moved on the sheet: C158, C219, C221, C223, C231, C233, C236, C237, C240, C241, C242, C244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

Commit message: Layout update
Layout with OP
Parts:
- U105, U108, U111, U94: footprint qaxe:BM1366 -> bitvein:BM1366
Changed lines of the file:
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@@
 			)
 		)
-		(property "Footprint" "qaxe:BM1366"
+		(property "Footprint" "bitvein:BM1366"
 			(at 327.66 76.2 0)
 			(effects
@@
 			)
 		)
-		(property "Footprint" "qaxe:BM1366"
+		(property "Footprint" "bitvein:BM1366"
 			(at 165.1 76.2 0)
 			(effects
@@
 			)
 		)
-		(property "Footprint" "qaxe:BM1366"
+		(property "Footprint" "bitvein:BM1366"
 			(at 83.82 76.2 0)
 			(effects
@@
 			)
 		)
-		(property "Footprint" "qaxe:BM1366"
+		(property "Footprint" "bitvein:BM1366"
 			(at 246.38 76.2 0)
 			(effects

Commit message: fixed level shifter, added optional headers for future extensions
Parts:
- U105, U108, U111, U94: footprint bitvein:BM1366 -> myfootprints:BM1366-user1-soldermask
Changed lines of the file:
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@@
 			)
 		)
-		(property "Footprint" "bitvein:BM1366"
+		(property "Footprint" "myfootprints:BM1366-user1-soldermask"
 			(at 327.66 76.2 0)
 			(effects
@@
 			)
 		)
-		(property "Footprint" "bitvein:BM1366"
+		(property "Footprint" "myfootprints:BM1366-user1-soldermask"
 			(at 165.1 76.2 0)
 			(effects
@@
 			)
 		)
-		(property "Footprint" "bitvein:BM1366"
+		(property "Footprint" "myfootprints:BM1366-user1-soldermask"
 			(at 83.82 76.2 0)
 			(effects
@@
 			)
 		)
-		(property "Footprint" "bitvein:BM1366"
+		(property "Footprint" "myfootprints:BM1366-user1-soldermask"
 			(at 246.38 76.2 0)
 			(effects
