File: 0xaxe/flex4.kicad_sch (KiCad schematic)
At the start: 89 parts, among them U10 +0V8, U11 +0V8, U12 +0V8, U13 +0V8, U14 +0V8, U15 +0V8, U16 +0V8, U17 +0V8, U18 +0V8, U19 BM1366_mode1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

Commit message: rev1.2
Connections:
- net +5V renamed +6.5V
Changed lines of the file:
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@@
 	)
 	(symbol
+		(lib_id "mylib7:+6.5V")
+		(at 83.82 186.69 0)
+		(unit 1)
+		(exclude_from_sim no)
+		(in_bom yes)
+		(on_board yes)
+		(dnp no)
+		(fields_autoplaced yes)
+		(property "Reference" "#PWR0272"
+			(at 83.82 190.5 0)
+			(effects
+				(font
+					(size 1.27 1.27)
+				)
+				(hide yes)
+			)
+		)
+		(property "Value" "+6.5V"
+			(at 83.82 181.61 0)
+			(effects
+				(font
+					(size 1.27 1.27)
+				)
+			)
+		)
+		(property "Footprint" ""
+			(at 83.82 186.69 0)
+			(effects
+				(font
+					(size 1.27 1.27)
+				)
+				(hide yes)
+			)
+		)
+		(property "Datasheet" ""
+			(at 83.82 186.69 0)
+			(effects
+				(font
+					(size 1.27 1.27)
+				)
+				(hide yes)
+			)
+		)
+		(property "Description" ""
+			(at 83.82 186.69 0)
+			(effects
+				(font
+					(size 1.27 1.27)
+				)
+				(hide yes)
+			)
+		)
+		(pin "1"
+		)
+		(instances
+			(project "0xaxe"
+				(path "/e63e39d7-6ac0-4ffd-8aa3-1841a4541b55/84d407d0-bd71-403d-bc5c-679b63d0a5ac/b5ee74d3-5a7e-48bf-a35d-6eb8d45bfd6b"
+					(reference "#PWR0272")
+					(unit 1)
+				)
+			)
+		)
+	)
+	(symbol
 		(lib_id "power:GND")
 		(at 270.51 194.31 0)
@@
 					(unit 1)
 				)
-			)
-		)
-	)
-	(symbol
-		(lib_id "power:+5V")
-		(at 83.82 186.69 0)
-		(unit 1)
-		(exclude_from_sim no)
-		(in_bom yes)
-		(on_board yes)
-		(dnp no)
-		(fields_autoplaced yes)
-		(property "Reference" "#PWR0272"
-			(at 83.82 190.5 0)
-			(effects
-				(font
-					(size 1.27 1.27)
-				)
-				(hide yes)
-			)
-		)
-		(property "Value" "+5V"
-			(at 83.82 181.61 0)
-			(effects
-				(font
-					(size 1.27 1.27)
-				)
-			)
-		)
-		(property "Footprint" ""
-			(at 83.82 186.69 0)
-			(effects
-				(font
-					(size 1.27 1.27)
-				)
-				(hide yes)
-			)
-		)
-		(property "Datasheet" ""
-			(at 83.82 186.69 0)
-			(effects
-				(font
-					(size 1.27 1.27)
-				)
-				(hide yes)
-			)
-		)
-		(property "Description" "Power symbol creates a global label with name \"+5V\""
-			(at 83.82 186.69 0)
-			(effects
-				(font
-					(size 1.27 1.27)
-				)
-				(hide yes)
-			)
-		)
-		(pin "1"
-		)
-		(instances
-			(project "0xaxe"
-				(path "/e63e39d7-6ac0-4ffd-8aa3-1841a4541b55/84d407d0-bd71-403d-bc5c-679b63d0a5ac/b5ee74d3-5a7e-48bf-a35d-6eb8d45bfd6b"
-					(reference "#PWR0272")
-					(unit 1)
-				)

Commit message: push
Parts:
- U5: footprint Package_SO:SOIC-16_3.9x9.9mm_P1.27mm -> Package_SO:QSOP-16_3.9x4.9mm_P0.635mm; Manufacturer ADUM141E0BRZ-RL7 -> ADUM141D1BRQZ; OrderNr 505-ADUM141E0BRZ-RL7CT-ND -> ADUM141D1BRQZ-ND
Changed lines of the file:
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@@
 			)
 		)
-		(property "Footprint" "Package_SO:SOIC-16_3.9x9.9mm_P1.27mm"
+		(property "Footprint" "Package_SO:QSOP-16_3.9x4.9mm_P0.635mm"
 			(at 101.6 158.75 0)
 			(effects
@@
 			)
 		)
-		(property "Manufacturer" "ADUM141E0BRZ-RL7"
+		(property "Manufacturer" "ADUM141D1BRQZ"
 			(at 101.6 140.97 0)
 			(effects
@@
 			)
 		)
-		(property "OrderNr" "505-ADUM141E0BRZ-RL7CT-ND"
+		(property "OrderNr" "ADUM141D1BRQZ-ND"
 			(at 101.6 140.97 0)
 			(effects
