File: 0xaxe/flex1.kicad_sch (KiCad schematic)
At the start: 89 parts, among them U115 MCP1824T-1802E, U5001 25MHz, U5003 NCP114ASN080T1G, U5004 ADUM141E0BRZ-RL7, U5005 +0V8, U5006 +0V8, U5007 BM1366_mode1, U5008 +0V8, U5009 +0V8, U5010 +0V8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

Commit message: push
Parts:
- U5004: footprint Package_SO:SOIC-16_3.9x9.9mm_P1.27mm -> Package_SO:QSOP-16_3.9x4.9mm_P0.635mm; Manufacturer ADUM141E0BRZ-RL7 -> ADUM141D1BRQZ; OrderNr 505-ADUM141E0BRZ-RL7CT-ND -> ADUM141D1BRQZ-ND
Changed lines of the file:
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@@
 			)
 		)
-		(property "Footprint" "Package_SO:SOIC-16_3.9x9.9mm_P1.27mm"
+		(property "Footprint" "Package_SO:QSOP-16_3.9x4.9mm_P0.635mm"
 			(at 105.41 157.48 0)
 			(effects
@@
 			)
 		)
-		(property "Manufacturer" "ADUM141E0BRZ-RL7"
+		(property "Manufacturer" "ADUM141D1BRQZ"
 			(at 105.41 139.7 0)
 			(effects
@@
 			)
 		)
-		(property "OrderNr" "505-ADUM141E0BRZ-RL7CT-ND"
+		(property "OrderNr" "ADUM141D1BRQZ-ND"
 			(at 105.41 139.7 0)
 			(effects
