File: 0xaxe/flex2.kicad_sch (KiCad schematic)
At the start: 89 parts, among them U14 MCP1824T-1802E, U6001 25MHz, U6003 NCP114ASN080T1G, U6004 ADUM141E0BRZ-RL7, U6005 +0V8, U6006 +0V8, U6007 BM1366_mode1, U6008 +0V8, U6009 +0V8, U6010 +0V8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

Commit message: push
Parts:
- U6004: footprint Package_SO:SOIC-16_3.9x9.9mm_P1.27mm -> Package_SO:QSOP-16_3.9x4.9mm_P0.635mm; Manufacturer ADUM141E0BRZ-RL7 -> ADUM141D1BRQZ; OrderNr 505-ADUM141E0BRZ-RL7CT-ND -> ADUM141D1BRQZ-ND
Changed lines of the file:
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@@
 			)
 		)
-		(property "Footprint" "Package_SO:SOIC-16_3.9x9.9mm_P1.27mm"
+		(property "Footprint" "Package_SO:QSOP-16_3.9x4.9mm_P0.635mm"
 			(at 104.14 151.13 0)
 			(effects
@@
 			)
 		)
-		(property "Manufacturer" "ADUM141E0BRZ-RL7"
+		(property "Manufacturer" "ADUM141D1BRQZ"
 			(at 104.14 133.35 0)
 			(effects
@@
 			)
 		)
-		(property "OrderNr" "505-ADUM141E0BRZ-RL7CT-ND"
+		(property "OrderNr" "ADUM141D1BRQZ-ND"
 			(at 104.14 133.35 0)
 			(effects
